Commit message: Created Gazebo

File: description/robot_core.xacro (robot description, xacro)
@@ -61,4 +61,7 @@
         </xacro:inertial_cylinder>
     </link>
+    <gazebo reference="left_wheel">
+        <material>Gazebo/Blue</material>
+    </gazebo>
     <joint name= "right_wheel_joint" type= "continuous">
         <parent link = "base_link"/>
@@ -83,4 +86,7 @@
         </xacro:inertial_cylinder>
     </link>
+    <gazebo reference="right_wheel">
+        <material>Gazebo/Blue</material>
+    </gazebo>
     <joint name = "castor_wheel_joint" type="fixed">
         <parent link="chassis"/>
@@ -104,3 +110,8 @@
         </xacro:inertial_sphere>
     </link>
+    <gazebo reference="castor_wheel">
+        <material>Gazebo/Black</material>
+        <mu1 value="0.001"/>
+        <mu2 value="0.001"/>
+    </gazebo>
 </robot>
